File: elec/layout/default/veml7700.kicad_pcb (KiCad board)
At the start: 2 copper layers, 225.7 x 100.8 mm, 0 parts

Commit message: added layout
Parts:
- added C1: 50V 100nF X7R ±10% 0603 Multilayer Ceramic Capacitors MLCC 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, lib:C0603, F.Cu at (243.8, 100.2)
- added U1: , lib:SENSOR-SMD_EML7700-TT, F.Cu at (243.8, 98.0)
Routing:
- net vcc: track 0.00 -> 2.31 mm
- net ic-gnd: track 0.00 -> 2.29 mm
Changed lines of the file:
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@@
   )
   (net 0 "")
+  (net 1 "scl")
+  (net 2 "vcc")
+  (net 3 "ic-gnd")
+  (net 4 "sda")
+  (footprint "lib:C0603" (layer "F.Cu")
+    (at 243.8 100.2)
+    (descr "Capacitor SMD 0603 (1608 Metric), square (rectangular) end terminal, IPC_7351 nominal, (Body size source: IPC-SM-782 page 76, https://www.pcb-3d.com/wordpress/wp-content/uploads/ipc-sm-782a_amendment_1_and_2.pdf), generated with kicad-footprint-generator")
+    (tags "capacitor")
+    (attr smd)
+    (fp_text reference "C1" (at 4.775 0) (layer "F.SilkS")
+        (effects (font (size 1 1) (thickness 0.15)))
+    )
+    (fp_text value "50V 100nF X7R ±10% 0603  Multilayer Ceramic Capacitors MLCC - SMD/SMT ROHS" (at 0 1.43) (layer "F.Fab")
+        (effects (font (size 1 1) (thickness 0.15)))
+    )
+    (fp_text user "${REFERENCE}" (at 0 0) (layer "F.Fab")
+        (effects (font (size 0.4 0.4) (thickness 0.06)))
+    )
+    (fp_line (start -0.14058 -0.51) (end 0.14058 -0.51)
+      (stroke (width 0.12) (type solid)) (layer "F.SilkS"))
+    (fp_line (start -0.14058 0.51) (end 0.14058 0.51)
+      (stroke (width 0.12) (type solid)) (layer "F.SilkS"))
+    (fp_line (start -1.48 -0.73) (end 1.48 -0.73)
+      (stroke (width 0.05) (type solid)) (layer "F.CrtYd"))
+    (fp_line (start -1.48 0.73) (end -1.48 -0.73)
+      (stroke (width 0.05) (type solid)) (layer "F.CrtYd"))
+    (fp_line (start 1.48 -0.73) (end 1.48 0.73)
+      (stroke (width 0.05) (type solid)) (layer "F.CrtYd"))
+    (fp_line (start 1.48 0.73) (end -1.48 0.73)
+      (stroke (width 0.05) (type solid)) (layer "F.CrtYd"))
+    (fp_line (start -0.8 -0.4) (end 0.8 -0.4)
+      (stroke (width 0.1) (type solid)) (layer "F.Fab"))
+    (fp_line (start -0.8 0.4) (end -0.8 -0.4)
+      (stroke (width 0.1) (type solid)) (layer "F.Fab"))
+    (fp_line (start 0.8 -0.4) (end 0.8 0.4)
+      (stroke (width 0.1) (type solid)) (layer "F.Fab"))
+    (fp_line (start 0.8 0.4) (end -0.8 0.4)
+      (stroke (width 0.1) (type solid)) (layer "F.Fab"))
+    (pad "1" smd roundrect (at -0.775 0) (size 0.9 0.95) (layers "F.Cu" "F.Paste" "F.Mask") (roundrect_rratio 0.25)
+      (net 2 "vcc") (pintype "stereo"))
+    (pad "2" smd roundrect (at 0.775 0) (size 0.9 0.95) (layers "F.Cu" "F.Paste" "F.Mask") (roundrect_rratio 0.25)
+      (net 3 "ic-gnd") (pintype "stereo"))
+    (model "${KICAD6_3DMODEL_DIR}/Capacitor_SMD.3dshapes/C_0603_1608Metric.wrl"
+      (offset (xyz 0 0 0))
+      (scale (xyz 1 1 1))
+      (rotate (xyz 0 0 0))
+    )
+  )
+  (footprint "lib:SENSOR-SMD_EML7700-TT" (layer "F.Cu")
+    (at 243.815 97.96)
+    (attr smd)
+    (fp_text reference "U1" (at 4.785 -0.36) (layer "F.SilkS")
+        (effects (font (size 1 1) (thickness 0.15)))
+    )
+    (fp_text value "" (at 0 4) (layer "F.Fab")
+        (effects (font (size 1 1) (thickness 0.15)))
+    )
+    (fp_text user "${REFERENCE}" (at 0 0) (layer "F.Fab")
+        (effects (font (size 1 1) (thickness 0.15)))
+    )
+    (fp_line (start -3.42 -2.54) (end -3.42 0.38)
+      (stroke (width 0.25) (type solid)) (layer "F.SilkS"))
+    (fp_line (start -3.42 -2.54) (end 3.43 -2.54)
+      (stroke (width 0.25) (type solid)) (layer "F.SilkS"))
+    (fp_line (start -3.42 0.38) (end -2.49 0.38)
+      (stroke (width 0.25) (type solid)) (layer "F.SilkS"))
+    (fp_line (start -1.32 0.38) (end -1.21 0.38)
+      (stroke (width 0.25) (type solid)) (layer "F.SilkS"))
+    (fp_line (start -0.05 0.38) (end 0.06 0.38)
+      (stroke (width 0.25) (type solid)) (layer "F.SilkS"))
+    (fp_line (start 1.22 0.38) (end 1.33 0.38)
+      (stroke (width 0.25) (type solid)) (layer "F.SilkS"))
+    (fp_line (start 2.49 0.38) (end 3.43 0.38)
+      (stroke (width 0.25) (type solid)) (layer "F.SilkS"))
+    (fp_line (start 3.43 0.38) (end 3.43 -2.54)
+      (stroke (width 0.25) (type solid)) (layer "F.SilkS"))
+    (fp_circle (center -2.92 -0.13) (end -2.74 -0.13)
+      (stroke (width 0.25) (type solid)) (fill none) (layer "F.SilkS"))
+    (fp_circle (center -2.41 0.89) (end -2.21 0.89)
+      (stroke (width 0.4) (type solid)) (fill none) (layer "Cmts.User"))
+    (fp_circle (center -3.4 0.46) (end -3.37 0.46)
+      (stroke (width 0.06) (type solid)) (fill none) (layer "F.Fab"))
+    (pad "1" smd rect (at -1.9 0) (size 0.7 1.6) (layers "F.Cu" "F.Paste" "F.Mask")
+      (net 1 "scl") (pintype "stereo"))
+    (pad "2" smd rect (at -0.63 0) (size 0.7 1.6) (layers "F.Cu" "F.Paste" "F.Mask")
+      (net 2 "vcc") (pintype "stereo"))
+    (pad "3" smd rect (at 0.63 0) (size 0.7 1.6) (layers "F.Cu" "F.Paste" "F.Mask")
+      (net 3 "ic-gnd") (pintype "stereo"))
+    (pad "4" smd rect (at 1.9 0) (size 0.7 1.6) (layers "F.Cu" "F.Paste" "F.Mask")
+      (net 4 "sda") (pintype "stereo"))
+    (model "/Users/nickk/projects/chess-clock/.ato/modules/smart-knob/.ato/modules/veml7700/elec/footprints/footprints.3dshapes/SENSOR-SMD_EML7700-TT.wrl"
+      (offset (xyz 0 1.04 -0))
+      (scale (xyz 1 1 1))
+      (rotate (xyz 0 0 0))
+    )
+  )
   (gr_circle (center 225.62 81.79) (end 227.32 81.79)
     (stroke (width 0.1) (type solid)) (fill none) (layer "Edge.Cuts"))
@@
       (xy 69.100734 49.778315)
     )
-    (stroke (width 0) (type solid)) (fill none) (layer "Edge.Cuts"))
+    (stroke (width 0.1) (type solid)) (fill none) (layer "Edge.Cuts"))
   (gr_arc (start 261.62 113.79) (mid 260.448427 116.618427) (end 257.62 117.79)
     (stroke (width 0.1) (type solid)) (layer "Edge.Cuts"))
@@
     (effects (font (size 2 2) (thickness 0.1)) (justify left bottom))
   )
+  (segment (start 243.185 97.96) (end 243.185 100.04) (width 0.25) (layer "F.Cu") (net 2))
+  (segment (start 243.185 100.04) (end 243.025 100.2) (width 0.25) (layer "F.Cu") (net 2))
+  (segment (start 244.445 100.07) (end 244.575 100.2) (width 0.25) (layer "F.Cu") (net 3))
+  (segment (start 244.445 97.96) (end 244.445 100.07) (width 0.25) (layer "F.Cu") (net 3))
   (group "" (id 6c1ef9f7-0f34-47bb-ac1a-76df23fb396e)
     (members
